File: X8-Backplane.sch (EAGLE design)
At the start: 15 parts, among them U1 BD6221FSOP, U2 MIC29501-5.0WU, U3 MIC29501-5.0WU

Commit message: first draft of the sechematic. Almost there!
Parts:
- removed U$2: BD6221, HBridge:BD6221
- added U$5: AP2210, PowerComponents:AP2210
- added U4, U5: FQB27P06, CamSensComponents:FQB27P06
Connections:
- removed net N$4: PCB1.3V3@1
- new net !RE: PCB1.GPIO23, U$1.!RE
- new net 3.3V: U$1.VCC13, U$1.VCC14, U$3.VIN, U$5.VOUT, U$7.VDDA, U$7.VDDB
- new net 3V3_PIEZO: U$4G$1.10, U$4G$1.9, U1.OUT1
- new net A: U$1.A, U$4G$1.25
- new net B: U$1.B, U$4G$1.23
- new net DE: PCB1.GPIO24, U$1.DE
- new net DSCLM: U$4G$1.35, U$7.DSCLM
- new net DSCLP: U$4G$1.36, U$7.DSCLP
- new net DSDAM: U$4G$1.37, U$7.DSDAM
- new net DSDAP: U$4G$1.38, U$7.DSDAP
- new net FIN: PCB1.GPIO13, U1.FIN
- new net GND_PIEZO: U$4G$1.11, U$4G$1.12, U1.OUT2
- new net LASER_5V: U$4G$2.17, U$4G$2.18, U5.D2
- new net LASER_ON: PCB1.GPIO5, U5.G2
- new net LED_5V: U$4G$2.19, U$4G$2.20, U4.D2
- new net LED_ON: PCB1.GPIO6, U4.G2
- new net RIN: U1.RIN
- new net RX: PCB1.GPIO15, U$1.R0
- new net SCL: PCB1.GPIO3, U$3.SCL, U$4G$1.40, U$7.SCL
- new net SDA: PCB1.GPIO2, U$3.SDA, U$4G$1.39, U$7.SDA
- new net SERVO_PWM: PCB1.GPIO18, U$4G$1.29
- new net TX: PCB1.GPIO14, U$1.DI
- new net Y: U$1.Y, U$4G$1.19
- new net Z: U$1.Z, U$4G$1.21
- net +12V: now also U$4G$2.26, U$4G$2.27, U$4G$2.28, U1.VCC@2, U1.VCC@3, U1.VREF
- net +5V: now also PCB1.5V@2, PCB1.5V@4, U$5.VIN; no longer U$4G$2.19, U$4G$2.20, U$4G$2.21, U$4G$2.22
- net +5V_CAMERA_TUBE: now also U$4G$2.13, U$4G$2.14, U$4G$2.15, U$4G$2.16, U4.S2, U5.S2; no longer U$4G$2.25, U$4G$2.26, U$4G$2.27, U$4G$2.28
- net GND: now also PCB1.GND@14, PCB1.GND@20, PCB1.GND@25, PCB1.GND@30, PCB1.GND@34, PCB1.GND@39, PCB1.GND@6, PCB1.GND@9, U$1.GND6, U$1.GND7, U$3.GND, U$4G$2.1, U$4G$2.10, U$4G$2.2, U$4G$2.3, U$4G$2.4, U$4G$2.5, U$4G$2.6, U$4G$2.7, U$4G$2.8, U$4G$2.9, U$5.GND, U$7.GND, U1.GND
Other:
- note added: "LASER"
- note added: "LED"
- moved on the sheet: U1
