File: X8-Backplane.sch (EAGLE design)
At the start: 54 parts, among them U1 BD6221FSOP, U4 FQB27P06, U5 FQB27P06, U6 FQB27P06, U7 LM2678

Commit message: added snorlax!
Parts:
- C3: device SparkFun-Capacitors:CAP0805 -> SparkFun-Capacitors:0.18UF-0603-10V-10%
- R10, R6, R7, R9: value (none) -> 10k
Changed lines of the file:
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@@
 <part name="U$2" library="PowerComponents" deviceset="SWITCHMODE_SCHOTTKY" device=""/>
 <part name="U7" library="PowerComponents" deviceset="LM2678" device=""/>
-<part name="C3" library="SparkFun-Capacitors" deviceset="CAP" device="0805" value="0.47uF"/>
 <part name="C4" library="SparkFun-Passives" deviceset="CAP" device="0603-CAP" value="0.01uF"/>
 <part name="GND17" library="SparkFun-Aesthetics" deviceset="GND" device=""/>
@@
 <part name="GND20" library="supply1" deviceset="GND" device=""/>
 <part name="GND21" library="supply1" deviceset="GND" device=""/>
-<part name="R6" library="SparkFun-Passives" deviceset="RESISTOR" device="0603-RES"/>
+<part name="R6" library="SparkFun-Passives" deviceset="RESISTOR" device="0603-RES" value="10k"/>
 <part name="SUPPLY5" library="SparkFun-Aesthetics" deviceset="3.3V" device=""/>
 <part name="SUPPLY6" library="SparkFun-Aesthetics" deviceset="3.3V" device=""/>
 <part name="C1" library="SparkFun-Capacitors" deviceset="0.1UF-25V(+80/-20%)(0603)" device="" value="0.1uF"/>
 <part name="GND22" library="supply1" deviceset="GND" device=""/>
-<part name="R7" library="SparkFun-Passives" deviceset="RESISTOR" device="0603-RES"/>
+<part name="R7" library="SparkFun-Passives" deviceset="RESISTOR" device="0603-RES" value="10k"/>
 <part name="GND23" library="supply1" deviceset="GND" device=""/>
 <part name="SUPPLY7" library="SparkFun-Aesthetics" deviceset="3.3V" device=""/>
 <part name="SUPPLY8" library="SparkFun-Aesthetics" deviceset="3.3V" device=""/>
-<part name="R9" library="SparkFun-Passives" deviceset="RESISTOR" device="0603-RES"/>
+<part name="R9" library="SparkFun-Passives" deviceset="RESISTOR" device="0603-RES" value="10k"/>
 <part name="SUPPLY9" library="SparkFun-Aesthetics" deviceset="3.3V" device=""/>
 <part name="SUPPLY10" library="SparkFun-Aesthetics" deviceset="3.3V" device=""/>
-<part name="R10" library="SparkFun-Passives" deviceset="RESISTOR" device="0603-RES"/>
+<part name="R10" library="SparkFun-Passives" deviceset="RESISTOR" device="0603-RES" value="10k"/>
 <part name="C5" library="SparkFun-Capacitors" deviceset="0.1UF-25V(+80/-20%)(0603)" device="" value="1uF"/>
 <part name="GND24" library="supply1" deviceset="GND" device=""/>
@@
 <part name="V+_ESC5" library="SparkFun-Connectors" deviceset="BANANA_CONN" device=""/>
 <part name="V+_ESC1" library="SparkFun-Connectors" deviceset="BANANA_CONN" device=""/>
+<part name="C3" library="SparkFun-Capacitors" deviceset="0.18UF" device="-0603-10V-10%" value="0.47uF"/>
 </parts>
 <sheets>
 <sheet>
 <plain>
-<text x="480.06" y="190.5" size="3.81" layer="91">LED</text>
-<text x="528.32" y="190.5" size="3.81" layer="91">LASER</text>
-<text x="508" y="137.16" size="3.81" layer="91">BLUE TOOTH LED</text>
-<text x="350.52" y="-15.24" size="5.08" layer="91">debugging pins</text>
-<text x="297.18" y="-7.62" size="1.778" layer="91">power pins</text>
-<text x="299.72" y="-55.88" size="1.778" layer="91">data pins</text>
+<text x="480.06" y="190.5" size="3.81" layer="97">LED</text>
+<text x="528.32" y="190.5" size="3.81" layer="97">LASER</text>
+<text x="508" y="137.16" size="3.81" layer="97">BLUE TOOTH LED</text>
+<text x="350.52" y="-15.24" size="5.08" layer="97">debugging pins</text>
+<text x="297.18" y="-7.62" size="1.778" layer="97">power pins</text>
+<text x="299.72" y="-55.88" size="1.778" layer="97">data pins</text>
 </plain>
 <instances>
@@
 </instance>
 <instance part="U7" gate="G$1" x="101.6" y="-142.24"/>
-<instance part="C3" gate="G$1" x="78.74" y="-147.32" smashed="yes">
-<attribute name="NAME" x="80.264" y="-144.399" size="1.778" layer="95"/>
-<attribute name="VALUE" x="80.264" y="-149.479" size="1.778" layer="96"/>
-</instance>
 <instance part="C4" gate="G$1" x="132.08" y="-134.62" smashed="yes" rot="R90">
 <attribute name="NAME" x="128.016" y="-132.461" size="1.778" layer="95" rot="R180"/>
@@
 <instance part="GND20" gate="1" x="78.74" y="-33.02"/>
 <instance part="GND21" gate="1" x="142.24" y="-78.74"/>
-<instance part="R6" gate="G$1" x="88.9" y="-81.28"/>
+<instance part="R6" gate="G$1" x="88.9" y="-81.28" smashed="yes">
+<attribute name="NAME" x="85.09" y="-79.7814" size="1.778" layer="95"/>
+<attribute name="VALUE" x="90.17" y="-79.502" size="1.778" layer="96"/>
+</instance>
 <instance part="SUPPLY5" gate="G$1" x="78.74" y="-81.28"/>
 <instance part="SUPPLY6" gate="G$1" x="152.4" y="-81.28"/>
 <instance part="C1" gate="G$1" x="147.32" y="-91.44"/>
 <instance part="GND22" gate="1" x="147.32" y="-99.06"/>
-<instance part="R7" gate="G$1" x="144.78" y="-50.8"/>
+<instance part="R7" gate="G$1" x="144.78" y="-50.8" smashed="yes">
+<attribute name="NAME" x="140.97" y="-49.3014" size="1.778" layer="95"/>
+<attribute name="VALUE" x="146.05" y="-49.022" size="1.778" layer="96"/>
+</instance>
 <instance part="GND23" gate="1" x="157.48" y="-55.88"/>
 <instance part="SUPPLY7" gate="G$1" x="144.78" y="-30.48"/>
 <instance part="SUPPLY8" gate="G$1" x="91.44" y="-35.56"/>
-<instance part="R9" gate="G$1" x="91.44" y="-45.72"/>
+<instance part="R9" gate="G$1" x="91.44" y="-45.72" smashed="yes">
+<attribute name="NAME" x="87.63" y="-44.2214" size="1.778" layer="95"/>
+<attribute name="VALUE" x="92.71" y="-43.942" size="1.778" layer="96"/>
+</instance>
 <instance part="SUPPLY9" gate="G$1" x="81.28" y="-45.72"/>
 <instance part="SUPPLY10" gate="G$1" x="81.28" y="-50.8"/>
-<instance part="R10" gate="G$1" x="91.44" y="-50.8"/>
+<instance part="R10" gate="G$1" x="91.44" y="-50.8" smashed="yes">
+<attribute name="NAME" x="87.63" y="-49.3014" size="1.778" layer="95"/>
+<attribute name="VALUE" x="92.71" y="-49.022" size="1.778" layer="96"/>
+</instance>
 <instance part="C5" gate="G$1" x="66.04" y="-45.72"/>
 <instance part="GND24" gate="1" x="66.04" y="-53.34"/>
@@
 <instance part="V+_ESC5" gate="G$1" x="358.14" y="-40.64"/>
 <instance part="V+_ESC1" gate="G$1" x="358.14" y="-50.8"/>
+<instance part="C3" gate="G$1" x="78.74" y="-147.32"/>
 </instances>
 <busses>
@@
 <wire x1="96.52" y1="-157.48" x2="104.14" y2="-157.48" width="0.1524" layer="91"/>
 <junction x="104.14" y="-157.48"/>
-<pinref part="C3" gate="G$1" pin="2"/>
 <wire x1="78.74" y1="-149.86" x2="78.74" y2="-157.48" width="0.1524" layer="91"/>
 <wire x1="78.74" y1="-157.48" x2="96.52" y2="-157.48" width="0.1524" layer="91"/>
@@
 <wire x1="58.42" y1="-149.86" x2="58.42" y2="-157.48" width="0.1524" layer="91"/>
 <junction x="58.42" y="-157.48"/>
+<pinref part="C3" gate="G$1" pin="2"/>
 </segment>
 <segment>
@@
 <wire x1="83.82" y1="-139.7" x2="78.74" y2="-139.7" width="0.1524" layer="91"/>
 <wire x1="78.74" y1="-139.7" x2="68.58" y2="-139.7" width="0.1524" layer="91"/>
-<pinref part="C3" gate="G$1" pin="1"/>
 <wire x1="68.58" y1="-139.7" x2="63.5" y2="-139.7" width="0.1524" layer="91"/>
 <wire x1="78.74" y1="-142.24" x2="78.74" y2="-139.7" width="0.1524" layer="91"/>
@@
 <wire x1="58.42" y1="-142.24" x2="58.42" y2="-139.7" width="0.1524" layer="91"/>
 <junction x="58.42" y="-139.7"/>
+<pinref part="C3" gate="G$1" pin="1"/>
 </segment>
 <segment>
@@
 <pinref part="U5" gate="G$1" pin="S2"/>
 <wire x1="538.48" y1="177.8" x2="538.48" y2="185.42" width="0.1524" layer="91"/>
-<label x="528.32" y="185.42" size="1.778" layer="95"/>
 <pinref part="RPI+5V2" gate="1" pin="+5V"/>
 </segment>
@@
 <pinref part="U4" gate="G$1" pin="S2"/>
 <wire x1="487.68" y1="177.8" x2="487.68" y2="185.42" width="0.1524" layer="91"/>
-<label x="477.52" y="185.42" size="1.778" layer="95"/>
 <pinref part="RPI+5V3" gate="1" pin="+5V"/>
 </segment>
@@
 <pinref part="U4" gate="G$1" pin="D2"/>
 <wire x1="487.68" y1="160.02" x2="487.68" y2="157.48" width="0.1524" layer="91"/>
-<label x="485.14" y="147.32" size="1.778" layer="95"/>
+<label x="480.06" y="147.32" size="1.778" layer="95"/>
 <pinref part="R5" gate="G$1" pin="2"/>
 <wire x1="487.68" y1="157.48" x2="487.68" y2="149.86" width="0.1524" layer="91"/>
